File: PCB/piano.kicad_sch (KiCad schematic)
At the start: 29 parts, among them J1 Conn_01x02, J2 Conn_01x04, J3 Conn_01x04, U1 WeMos_D1_mini

Commit message: v0.2 PCB
Parts:
- added J4: Conn_01x02, Connector_JST:JST_EH_B2B-EH-A_1x02_P2.50mm_Vertical, symbol Connector_Generic:Conn_01x02
- added Q1: 2N3904, Package_TO_SOT_THT:TO-92_Inline, symbol Transistor_BJT:2N3904
- added R5: 10k, Resistor_SMD:R_1206_3216Metric_Pad1.30x1.75mm_HandSolder, symbol Device:R
- added SW1: SW_SPDT_MSM, Suat:Schiebeschalter, symbol Switch:SW_SPDT_MSM
- added U2: LiPo_Module, Suat:LiPoChargerModule, symbol Suat:LiPo_Module
- R1, R2, R3, R4: value R -> 10k
- SW-0: value SW_Push -> 0x0
- SW-1: value SW_Push -> 0x1
- SW-2: value SW_Push -> 0x2
- SW-3: value SW_Push -> 0x3
- SW-4: value SW_Push -> 0x4
- SW-5: value SW_Push -> 0x5
- SW-6: value SW_Push -> 0x6
- SW-7: value SW_Push -> 0x7
- SW-8: value SW_Push -> 0x8
- SW-9: value SW_Push -> 0x9
- SW-A1: renamed from SW-A; value SW_Push -> 0xA
- SW-B1: renamed from SW-B; value SW_Push -> 0xB
- SW-C1: renamed from SW-C; value SW_Push -> 0xC
- SW-D1: renamed from SW-D; value SW_Push -> 0xD
- SW-E1: renamed from SW-E; value SW_Push -> 0xE3
- SW-F1: renamed from SW-F; value SW_Push -> 0xF
Connections:
- net GND: now also J4.2 (Pin_2), Q1.1 (E), U2.1 (GND), U2.3 (GND); no longer BZ1.2 (+), J1.1 (Pin_1)
- net at U1.3 (D0): now also R5.1; no longer BZ1.1 (-)
- net at U1.9 (5V): now also BZ1.1 (-), SW1.1; no longer J1.2 (Pin_2)
- new net: Q1.2 (B), R5.2
- new net: BZ1.2 (+), Q1.3 (C)
- new net: SW1.2, U2.6 (VOUT)
- new net: J4.1 (Pin_1), U2.2 (VIN)
- new net: J1.2 (Pin_2), U2.4 (B-)
- new net: J1.1 (Pin_1), U2.5 (B+)
Other:
- moved on the sheet: BZ1, J1, U1

Commit message: update pcb (larger footprint for transistor)
Parts:
- added H1: MountingHole, symbol Mechanical:MountingHole
Changed lines of the file:
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@@
     (pin "2")
+  )
+  (symbol (lib_id "Mechanical:MountingHole") (at 34.29 160.02 0) (unit 1)
+    (in_bom yes) (on_board yes) (fields_autoplaced)
+    (property "Reference" "H1" (id 0) (at 36.83 158.7499 0)
+      (effects (font (size 1.27 1.27)) (justify left))
+    )
+    (property "Value" "MountingHole" (id 1) (at 36.83 161.2899 0)
+      (effects (font (size 1.27 1.27)) (justify left))
+    )
+    (property "Footprint" "" (id 2) (at 34.29 160.02 0)
+      (effects (font (size 1.27 1.27)) hide)
+    )
+    (property "Datasheet" "~" (id 3) (at 34.29 160.02 0)
+      (effects (font (size 1.27 1.27)) hide)
+    )
   )
   (symbol (lib_id "power:GND") (at 261.62 63.5 0) (unit 1)
@@
       (reference "D4") (unit 1) (value "DIODE") (footprint "Diode_SMD:D_0805_2012Metric")
     )
+    (path "/802bd717-75a4-4efc-bdc3-ab512c6bce65"
+      (reference "H1") (unit 1) (value "MountingHole") (footprint "")
+    )
     (path "/a95ec438-937f-42fa-893e-a9983fa0e648"
